Commit message: updated hardware representation urdf to match current hardware, and modified the launch file just to display the urdf model!

File: urdf/first_hardware_representation.urdf (robot description, URDF)
Before this commit: robot Transporter_model_1.0, 6 links, 5 joints
Links:
- removed link us_front_link
- removed link us_left_link
- removed link us_right_link
- added link top_sensor_layer; visual box size=0.5 0.5 0.0045
- added link us_front; visual mesh filename=package://robot_model_test/meshes/HC-SR04-binary.stl scale=0.001 0.001 0.001
- added link us_left; visual mesh filename=package://robot_model_test/meshes/HC-SR04-binary.stl scale=0.001 0.001 0.001
- added link us_right; visual mesh filename=package://robot_model_test/meshes/HC-SR04-binary.stl scale=0.001 0.001 0.001
- link base_link: geometry visual box size=0.5 0.5 0.4735
Joints:
- added joint top_sensor_layer_joint: type fixed, parent base_link, child top_sensor_layer, origin xyz=0 0 0.478
- joint camera_joint: origin xyz=0.27 0 0.3 -> xyz=0.23315 0 -0.03615; parent base_link -> top_sensor_layer
- joint lidar_joint: origin xyz=0 0 0.40146 -> xyz=0 0 0.06246; parent base_link -> top_sensor_layer
- joint us_front_joint: child us_front_link -> us_front; origin xyz=0.255 0 0.381 rpy=0 0 0 -> xyz=0.255 0 0.04 rpy=0 0 0; parent base_link -> top_sensor_layer
- joint us_left_joint: child us_left_link -> us_left; origin xyz=0.219 0.219 0.381 rpy=0 0 0.78539 -> xyz=0.219 0.219 0.04 rpy=0 0 0.78539; parent base_link -> top_sensor_layer
- joint us_right_joint: child us_right_link -> us_right; origin xyz=0.219 -0.219 0.381 rpy=0 0 -0.78539 -> xyz=0.219 -0.219 0.04 rpy=0 0 -0.78539; parent base_link -> top_sensor_layer
